File: hhkb.kicad_pcb (KiCad board)
At the start: 2 copper layers, 285 x 100 mm, 147 parts, among them J1 Conn_01x04_MountingPin, SW1 SW_Push, U1 ATmega32U4-MU, Y1 16MHz

Commit message: updates
Parts:
- added C14: 0.1uF, Capacitor_SMD:C_0805_2012Metric, B.Cu at (110.6, 81.6)
- added C15: 0.1uF, Capacitor_SMD:C_0805_2012Metric, B.Cu at (99.7, 81.3)
- added D12: D_Small, Diode_SMD:D_SOD-123, B.Cu at (27.8, 79.8)
- added LED6: WS2812B, WS2812B:WS2812BDual, F.Cu at (110.6, 87.1)
- added LED7: WS2812B, WS2812B:WS2812BDual, F.Cu at (99.6, 87.1)
- added SW_LCTRL2: MX-NoLED, MX_NEC:mx-nec-alps, F.Cu at (18.2, 86.9)
- moved R1 90.1 mm to (253.0, 86.5)
- moved C1 88.5 mm to (254.1, 79.5)
- moved C4 88.5 mm to (272.2, 81.5)
- moved C5 88.5 mm to (267.2, 95.9)
- moved C7 88.5 mm to (269.3, 95.9)
- moved U1 88.5 mm to (262.3, 86.8)
- moved C2 88.5 mm to (271.3, 95.9)
- moved C3 88.5 mm to (272.6, 89.4)
- moved Y1 88.5 mm to (271.9, 86.3)
- moved C6 87.3 mm to (261.6, 77.1)
- moved R4 86.3 mm to (253.7, 93.3)
- moved R3 83.9 mm to (276.8, 83.0)
- moved SW1 79.4 mm to (279.5, 95.9), turned to 180 degrees
- moved C12 54.8 mm to (156.0, 81.9)
- moved C10 54.8 mm to (178.1, 81.7)
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Connections:
- LED5 pad 2: unconnected-(LED5-DOUT) -> Net-(LED5-DOUT)
- SW_B1 pad 1: COL2 -> COL3
- SW_C1 pad 1: COL1 -> COL2
- SW_J1 pad 1: COL3 -> COL4
- SW_PERIOD1 pad 1: COL4 -> COL5
- SW_RSH1 pad 1: COL5 -> COL6
- SW_Z1 pad 1: COL0 -> COL1
- U1 pad 10: ROW8 -> unconnected-(U1-PB2-Pad10)
- U1 pad 11: ROW0 -> COL6
- U1 pad 12: ROW2 -> unconnected-(U1-PB7-Pad12)
- U1 pad 18: ROW5 -> unconnected-(U1-PD0-Pad18)
- U1 pad 19: unconnected-(U1-PD1) -> ROW0
- U1 pad 20: unconnected-(U1-PD2) -> ROW3
- U1 pad 21: ROW3 -> ROW8
- U1 pad 25: ROW4 -> COL0
- U1 pad 26: unconnected-(U1-PD6) -> COL1
- U1 pad 27: unconnected-(U1-PD7) -> COL2
- U1 pad 28: unconnected-(U1-PB4) -> COL3
- U1 pad 29: COL6 -> COL4
- U1 pad 36: COL1 -> ROW6
- U1 pad 37: COL0 -> ROW2
- U1 pad 38: COL2 -> ROW1
- U1 pad 40: COL3 -> unconnected-(U1-PF1-Pad40)
- U1 pad 41: COL4 -> ROW5
- U1 pad 8: ROW6 -> unconnected-(U1-PB0-Pad8)
- U1 pad 9: ROW1 -> ROW4
Routing:
- net COL2: track 196.2 -> 337.0 mm, vias 12 -> 8
- net COL3: track 165.4 -> 287.7 mm
- net COL0: track 338.0 -> 459.1 mm
- net COL1: track 283.5 -> 384.4 mm, vias 12 -> 10
- net COL6: track 271.2 -> 182.9 mm, vias 9 -> 8
- net Net-(U1-D-): track 127.4 -> 39.6 mm
- net Net-(U1-D+): track 124.6 -> 40.1 mm
- net BUZIN: track 31.3 -> 86.0 mm, vias 0 -> 4
- net COL4: track 200.3 -> 253.7 mm, vias 15 -> 11
- net ROW0: track 332.0 -> 379.2 mm, vias 8 -> 4
- net LEDDIN: track 41.2 -> 80.6 mm
- net ROW3: track 302.2 -> 340.3 mm, vias 16 -> 10
- net ROW5: track 281.3 -> 311.0 mm
- net Net-(LED4-DOUT): track 11.0 -> 37.0 mm
- net ROW2: track 320.0 -> 336.2 mm, vias 4 -> 2
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