File: hhkb.kicad_sch (KiCad schematic)
At the start: 147 parts, among them J1 Conn_01x04_MountingPin, SW1 SW_Push, U1 ATmega32U4-MU, Y1 16MHz

Commit message: updates
Parts:
- added C14, C15: 0.1uF, Capacitor_SMD:C_0805_2012Metric, symbol Device:C_Small
- added D12: D_Small, Diode_SMD:D_SOD-123, symbol Device:D_Small
- added LED6, LED7: WS2812B, WS2812B:WS2812BDual, symbol ws2812b:WS2812B
- added SW_LCTRL2: MX-NoLED, MX_NEC:mx-nec-alps, symbol MX_Alps_Hybrid:MX-NoLED
Connections:
- net +5V: now also C14.2, C15.2, LED6.1 (VCC), LED7.1 (VCC)
- net COL0: now also U1.25 (PD4), SW_LCTRL2.1 (COL); no longer SW_Z1.1 (COL), U1.37 (PF6)
- net COL1: now also SW_Z1.1 (COL), U1.26 (PD6); no longer SW_C1.1 (COL), U1.36 (PF7)
- net COL2: now also SW_C1.1 (COL), U1.27 (PD7); no longer SW_B1.1 (COL), U1.38 (PF5)
- net COL3: now also SW_B1.1 (COL), U1.28 (PB4); no longer SW_J1.1 (COL), U1.40 (PF1)
- net COL4: now also SW_J1.1 (COL), U1.29 (PB5); no longer SW_PERIOD1.1 (COL), U1.41 (PF0)
- net COL5: now also SW_PERIOD1.1 (COL); no longer SW_RSH1.1 (COL)
- net COL6: now also SW_RSH1.1 (COL), U1.11 (PB3); no longer U1.29 (PB5)
- net GND: now also C14.1, C15.1, LED6.3 (GND), LED7.3 (GND)
- net ROW0: now also U1.19 (PD1); no longer U1.11 (PB3)
- net ROW1: now also U1.38 (PF5); no longer U1.9 (PB1)
- net ROW2: now also U1.37 (PF6); no longer U1.12 (PB7)
- net ROW3: now also U1.20 (PD2); no longer U1.21 (PD3)
- net ROW4: now also U1.9 (PB1); no longer U1.25 (PD4)
- net ROW5: now also U1.41 (PF0), D12.1 (K); no longer U1.18 (PD0)
- net ROW6: now also U1.36 (PF7); no longer U1.8 (PB0)
- net ROW8: now also U1.21 (PD3); no longer U1.10 (PB2)
- net at LED5.2 (DOUT): now also LED6.4 (DIN)
- new net: LED6.2 (DOUT), LED7.4 (DIN)
- new net: D12.2 (A), SW_LCTRL2.2 (ROW)
Other:
- moved on the sheet: C10, C12, C13, C9, D18, D29, D40, D51, D62, D8, LED2, LED3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

Commit message: update
Parts:
- renumbered SW_F13 to SW_F1
Changed lines of the file:
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@@
   (symbol (lib_id "MX_Alps_Hybrid:MX-NoLED") (at 195.58 104.14 0) (unit 1)
     (in_bom yes) (on_board yes) (dnp no)
-    (property "Reference" "SW_F13" (at 196.4182 98.4758 0)
+    (property "Reference" "SW_F1" (at 196.4182 98.4758 0)
       (effects (font (size 1.524 1.524)))
     )
@@
       (project "hhkb"
         (path "/151da08b-0979-4785-a9bf-6fa9b165d629"
-          (reference "SW_F13") (unit 1)
+          (reference "SW_F1") (unit 1)
         )
       )
